File: master/ee/chest-xmega-rgb.brd (EAGLE design)
At the start: 164 x 146 mm, 104 parts, among them IC1 XMEGA-A3, IC3 XMEGA-A4, J1(RS) RJ11-6PTH, J2(LS) RJ11-6PTH, T1 2N2222, T2 2N2222, U1 LCD-16X2-G4, U2 TS5A63157

Commit message: chest board: drop in replace HUGE LEDs with SMT
Parts:
- RGB1, RGB2, RGB3, RGB4, RGB5, RGB6, RGB7, RGB8: value RGBLED -> AVAGO-RGB-SMT; device greg:RGB-LED-10MM-COMMON-ANODE -> greg:AVAGO-SMT-RGB
- turned RGB1 to 270 degrees
- turned RGB2 to 270 degrees
- turned RGB3 to 270 degrees
- turned RGB4 to 270 degrees
- turned RGB5 to 90 degrees
- turned RGB6 to 90 degrees
- turned RGB7 to 90 degrees
- turned RGB8 to 90 degrees
Connections:
- net +7V2: now also RGB1.P$4, RGB1.P$5, RGB1.P$6, RGB2.P$4, RGB2.P$5, RGB2.P$6, RGB4.P$4, RGB4.P$5, RGB4.P$6, RGB5.P$4, RGB5.P$5, RGB5.P$6, RGB6.P$4, RGB6.P$5, RGB6.P$6, RGB7.P$4, RGB7.P$5, RGB7.P$6, RGB8.P$4, RGB8.P$5, RGB8.P$6; no longer RGB1.3, RGB2.3, RGB3.3, RGB4.3, RGB5.3, RGB6.3, RGB7.3, RGB8.3
- net N$17: now also RGB7.P$1; no longer RGB7.1
- net N$24: now also RGB7.P$3; no longer RGB7.4
- net N$27: now also RGB7.P$2; no longer RGB7.2
- net N$31: now also RGB8.P$3; no longer RGB8.4
- net N$32: now also RGB8.P$2; no longer RGB8.2
- net N$33: now also RGB8.P$1; no longer RGB8.1
- net N$35: now also RGB5.P$3; no longer RGB5.4
- net N$36: now also RGB5.P$2; no longer RGB5.2
- net N$37: now also RGB5.P$1; no longer RGB5.1
- net N$38: now also RGB6.P$3; no longer RGB6.4
- net N$39: now also RGB6.P$2; no longer RGB6.2
- net N$40: now also RGB6.P$1; no longer RGB6.1
- net N$41: now also RGB1.P$3; no longer RGB1.4
- net N$42: now also RGB1.P$2; no longer RGB1.2
- net N$43: now also RGB1.P$1; no longer RGB1.1
- net N$48: now also RGB2.P$3; no longer RGB2.4
- net N$49: now also RGB2.P$2; no longer RGB2.2
- net N$50: now also RGB2.P$1; no longer RGB2.1
- net N$51: now also RGB4.P$3; no longer RGB4.4
- net N$52: now also RGB4.P$2; no longer RGB4.2
- net N$53: now also RGB4.P$1; no longer RGB4.1
- net N$54: now also RGB3.P$1; no longer RGB3.1
- net N$55: now also RGB3.P$2; no longer RGB3.2
- net N$56: now also RGB3.P$3; no longer RGB3.4
Routing:
- net +7V2: track 677.3 -> 587.3 mm
- net N$37: track 37.1 -> 0.00 mm
- net N$36: track 34.9 -> 0.00 mm
- net N$35: track 32.8 -> 0.00 mm
- net N$31: track 33.6 -> 29.4 mm
- net N$43: track 34.6 -> 32.1 mm
- net N$17: track 30.0 -> 28.4 mm
- net N$51: track 32.3 -> 30.9 mm
- net N$52: track 37.1 -> 36.0 mm
- net N$55: track 24.1 -> 23.2 mm
- net N$33: track 45.0 -> 44.4 mm
- net N$49: track 24.3 -> 23.6 mm
- net N$40: track 26.3 -> 25.7 mm
