File: master/ee/chest-xmega-rgb.sch (EAGLE design)
At the start: 104 parts, among them IC1 XMEGA-A3, IC3 XMEGA-A4, J1(RS) RJ11-6PTH, J2(LS) RJ11-6PTH, T1 2N2222, T2 2N2222, U1 LCD-16X2-G4, U2 TS5A63157, U3 AT45DB321D-SU

Commit message: chest board: drop in replace HUGE LEDs with SMT
Parts:
- RGB1, RGB2, RGB3, RGB4, RGB5, RGB6, RGB7, RGB8: value RGBLED -> AVAGO-RGB-SMT; device greg:RGBLED -> greg:AVAGO-RGB-SMT
Connections:
- net +7V2: no longer RGB3.VCC
- net N$17: now also RGB7.BLUE; no longer RGB7.B
- net N$24: now also RGB7.RED; no longer RGB7.R
- net N$27: now also RGB7.GREEN; no longer RGB7.G
- net N$31: now also RGB8.RED; no longer RGB8.R
- net N$32: now also RGB8.GREEN; no longer RGB8.G
- net N$33: now also RGB8.BLUE; no longer RGB8.B
- net N$35: now also RGB5.RED; no longer RGB5.R
- net N$36: now also RGB5.GREEN; no longer RGB5.G
- net N$37: now also RGB5.BLUE; no longer RGB5.B
- net N$38: now also RGB6.RED; no longer RGB6.R
- net N$39: now also RGB6.GREEN; no longer RGB6.G
- net N$40: now also RGB6.BLUE; no longer RGB6.B
- net N$41: now also RGB1.RED; no longer RGB1.R
- net N$42: now also RGB1.GREEN; no longer RGB1.G
- net N$43: now also RGB1.BLUE; no longer RGB1.B
- net N$48: now also RGB2.RED; no longer RGB2.R
- net N$49: now also RGB2.GREEN; no longer RGB2.G
- net N$50: now also RGB2.BLUE; no longer RGB2.B
- net N$51: now also RGB4.RED; no longer RGB4.R
- net N$52: now also RGB4.GREEN; no longer RGB4.G
- net N$53: now also RGB4.BLUE; no longer RGB4.B
- net N$54: now also RGB3.BLUE; no longer RGB3.B
- net N$55: now also RGB3.GREEN; no longer RGB3.G
- net N$56: now also RGB3.RED; no longer RGB3.R
